File: kinesis_fkeys/right_fkeys.kicad_sch (KiCad schematic)
At the start: 21 parts

Commit message: removed properties in schematics and updated kicad project version
Parts:
- gave numbers to parts that had none: 10
